File: pcbv3/bbotsv3.brd (EAGLE design)
At the start: 66 x 66 mm, 22 parts

Commit message: ready to manufacture, review done
Parts:
- D1: device adafruit:DO-1N4148 -> my-library:DO-1N4148
- moved D1 0.32 mm to (5.40, 46.7)
- renumbered E1 to BAT1
Other:
- outline, holes or cut-outs redrawn
- board text added: "12V"
- board text added: "BAT2"
- board text removed: "ARMA"
- board text removed: "E2"
Changed lines of the file:
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@@
 <drawing>
 <settings>
-<setting alwaysvectorfont="yes"/>
+<setting alwaysvectorfont="no"/>
 <setting verticaltext="up"/>
 </settings>
-<grid distance="12.5" unitdist="mil" unit="mil" style="lines" multiple="1" display="no" altdistance="5" altunitdist="mil" altunit="mil"/>
+<grid distance="12.5" unitdist="mil" unit="mil" style="lines" multiple="1" display="yes" altdistance="5" altunitdist="mil" altunit="mil"/>
 <layers>
 <layer number="1" name="Top" color="4" fill="1" visible="yes" active="yes"/>
@@
 </layers>
 <board>
-<fusionsync huburn="a.cGVyc29uYWw6dWUyYzRkOTA5" projecturn="a.cGVyc29uYWw6dWUyYjkxNGFhIzIwMjIwNzIyNTQxNDA4NzAx" f3durn="urn:adsk.wipprod:dm.lineage:LMK6uCyRSQKW0e5iuERoUA" pcbguid="" lastpulledtime="2023-03-29T23:28:58Z" lastsyncedchangeguid="" latestrevisionid="6c6256d0-1dc8-4dbf-9463-9ebba56debc9" lastsyncedrevisionid="6c6256d0-1dc8-4dbf-9463-9ebba56debc9" lastboardhashguid="97264ad9-789f-a25e-7ed8-5b0a31e148d4" lastpushedtime="2023-03-30T01:55:14Z" linktopcb3d="true"/>
+<fusionsync huburn="a.cGVyc29uYWw6dWUyYzRkOTA5" projecturn="a.cGVyc29uYWw6dWUyYjkxNGFhIzIwMjIwNzIyNTQxNDA4NzAx" f3durn="urn:adsk.wipprod:dm.lineage:LMK6uCyRSQKW0e5iuERoUA" pcbguid="" lastpulledtime="2023-04-03T15:19:18Z" lastsyncedchangeguid="" latestrevisionid="6653b62f-8249-401f-bf6c-fbf95e6828b3" lastsyncedrevisionid="6653b62f-8249-401f-bf6c-fbf95e6828b3" lastboardhashguid="a39438af-997a-7943-2ca0-8df0f8b6bbd3" lastpushedtime="2023-04-03T15:37:57Z" linktopcb3d="true"/>
 <plain>
 <text x="5.08" y="20.32" size="1.27" layer="21" rot="R90">Diseño por Leslie C.
@@
 <text x="60.96" y="8.255" size="1.27" layer="22" rot="MR90">Diseño por Leslie C.
 para Battlebots 2023-1</text>
-<hole x="3" y="3" drill="3.2"/>
-<hole x="62.175" y="3.9525" drill="3.2"/>
-<hole x="62.175" y="62.4925" drill="3.2"/>
-<wire x1="0" y1="3" x2="3" y2="0" width="0.1524" layer="20" curve="90"/>
-<wire x1="3" y1="0" x2="63" y2="0" width="0.1524" layer="20"/>
-<wire x1="63" y1="0" x2="66" y2="3" width="0.1524" layer="20" curve="90"/>
-<wire x1="66" y1="3" x2="66" y2="63" width="0.1524" layer="20"/>
-<wire x1="66" y1="63" x2="63" y2="66" width="0.1524" layer="20" curve="90"/>
-<wire x1="63" y1="66" x2="3" y2="66" width="0.1524" layer="20"/>
-<wire x1="3" y1="66" x2="0" y2="63" width="0.1524" layer="20" curve="90"/>
-<wire x1="0" y1="63" x2="0" y2="3" width="0.1524" layer="20"/>
-<text x="51.7525" y="62.5475" size="1.778" layer="21">ARMA</text>
+<text x="52.705" y="62.5475" size="1.778" layer="21">12V</text>
 <text x="41.275" y="62.5475" size="1.778" layer="21">MOT_B</text>
 <text x="31.115" y="62.5475" size="1.778" layer="21">MOT_A</text>
-<text x="22.5425" y="62.5475" size="1.778" layer="21">E2</text>
-<text x="19.05" y="62.5475" size="1.778" layer="21">+</text>
-<text x="26.67" y="62.5475" size="1.778" layer="21">-</text>
+<text x="20.6375" y="62.5475" size="1.778" layer="21">BAT2</text>
+<text x="18.415" y="62.5475" size="1.778" layer="21">+</text>
+<text x="27.305" y="62.5475" size="1.778" layer="21">-</text>
 <text x="3.175" y="63.1825" size="1.778" layer="21" rot="R90">+</text>
-<text x="3.175" y="53.6575" size="1.778" layer="21" rot="R90">-</text>
+<text x="3.175" y="54.2925" size="1.778" layer="21" rot="R90">-</text>
 <text x="50.4825" y="62.23" size="1.778" layer="21">+</text>
 <text x="58.1025" y="62.23" size="1.778" layer="21">-</text>
@@
 <text x="56.8325" y="36.83" size="1.016" layer="21">5V</text>
 <text x="56.8325" y="32.0675" size="1.016" layer="21">5V</text>
+<hole x="3" y="3" drill="3.2"/>
+<hole x="63" y="3" drill="3.2"/>
+<hole x="63" y="63" drill="3.2"/>
+<wire x1="0" y1="63" x2="0" y2="3" width="0.1524" layer="20"/>
+<wire x1="0" y1="3" x2="3" y2="0" width="0.1524" layer="20" curve="90.0001"/>
+<wire x1="3" y1="0" x2="63" y2="0" width="0.1524" layer="20"/>
+<wire x1="63" y1="0" x2="63.2615" y2="0.0114" width="0.1524" layer="20"/>
+<wire x1="63.2615" y1="0.0114" x2="66" y2="3" width="0.1524" layer="20" curve="85.0001"/>
+<wire x1="66" y1="3" x2="66" y2="63" width="0.1524" layer="20"/>
+<wire x1="66" y1="63" x2="65.9886" y2="63.2615" width="0.1524" layer="20"/>
+<wire x1="65.9886" y1="63.2615" x2="63" y2="66" width="0.1524" layer="20" curve="85.0001"/>
+<wire x1="63" y1="66" x2="3" y2="66" width="0.1524" layer="20"/>
+<wire x1="3" y1="66" x2="2.7385" y2="65.9886" width="0.1524" layer="20"/>
+<wire x1="2.7385" y1="65.9886" x2="0" y2="63" width="0.1524" layer="20" curve="85.0001"/>
 </plain>
 <attributes>
@@
 <attribute name="NAME" x="15.5575" y="16.1925" size="1.27" layer="25" rot="R180"/>
 </element>
-<element name="D1" library="adafruit" library_urn="urn:adsk.eagle:library:420" package="DO-1N4148" package3d_urn="urn:adsk.eagle:package:6240748/1" value="" x="5.3975" y="46.99" smashed="yes" rot="R270">
-<attribute name="NAME" x="4.7625" y="48.26" size="1.27" layer="25" rot="R270"/>
-<attribute name="VALUE" x="5.1435" y="49.022" size="0.6096" layer="21" rot="R270"/>
-</element>
 <element name="Q1" library="adafruit" library_urn="urn:adsk.eagle:library:420" package="SOT23-W" package3d_urn="urn:adsk.eagle:package:6240750/1" value="" x="45.085" y="20.32" smashed="yes" rot="R270">
 <attribute name="NAME" x="44.3865" y="24.3205" size="1.27" layer="25" rot="R270"/>
@@
 <element name="ARMA2" library="KF301-2P-Terminal" package="KF301-2P" value="TERMINAL_2P" x="44.45" y="58.42" smashed="yes"/>
 <element name="ARMA3" library="KF301-2P-Terminal" package="KF301-2P" value="TERMINAL_2P" x="23.495" y="58.42" smashed="yes"/>
-<element name="E1" library="con-phoenix-508" library_urn="urn:adsk.eagle:library:176" package="MSTBA2" package3d_urn="urn:adsk.eagle:package:9615/1" value="MSTBA2" x="9.2075" y="59.3725" smashed="yes" rot="R270">
+<element name="BAT1" library="con-phoenix-508" library_urn="urn:adsk.eagle:library:176" package="MSTBA2" package3d_urn="urn:adsk.eagle:package:9615/1" value="MSTBA2" x="9.2075" y="59.3725" smashed="yes" rot="R270">
 <attribute name="MF" value="FARNELL" x="9.2075" y="59.3725" size="1.778" layer="27" rot="R270" display="off"/>
 <attribute name="MPN" value="1757242" x="9.2075" y="59.3725" size="1.778" layer="27" rot="R270" display="off"/>
-<attribute name="NAME" x="1.5875" y="60.3885" size="1.778" layer="25" ratio="10" rot="R270"/>
+<attribute name="NAME" x="2.2225" y="59.3725" size="1.778" layer="25" ratio="10" rot="R270" align="center"/>
 <attribute name="OC_FARNELL" value="3705171" x="9.2075" y="59.3725" size="1.778" layer="27" rot="R270" display="off"/>
 <attribute name="OC_NEWARK" value="71C4161" x="9.2075" y="59.3725" size="1.778" layer="27" rot="R270" display="off"/>
 <attribute name="POPULARITY" value="11" x="9.2075" y="59.3725" size="1.778" layer="27" rot="R270" display="off"/>
 <attribute name="VALUE" x="9.2075" y="64.4525" size="1.778" layer="27" ratio="10" rot="R270"/>
+</element>
+<element name="D1" library="my-library" library_urn="urn:adsk.eagle:library:37248401" package="DO-1N4148" package3d_urn="urn:adsk.eagle:package:6240748/1" value="" x="5.3975" y="46.6725" smashed="yes" rot="R270">
+<attribute name="NAME" x="4.7625" y="47.9425" size="1.27" layer="25" rot="R270"/>
+<attribute name="VALUE" x="5.1435" y="48.7045" size="0.6096" layer="21" rot="R270"/>
 </element>
 </elements>
@@
 <contactref element="U$1" pad="IN+"/>
 <contactref element="U$3" pad="IN+"/>
-<wire x1="8.8425" y1="24.01875" x2="9.36625" y2="23.495" width="1.27" layer="1"/>
+<wire x1="7.46125" y1="25.4" x2="9.36625" y2="23.495" width="1.27" layer="1"/>
 <wire x1="9.36625" y1="23.495" x2="9.525" y2="23.495" width="0.8128" layer="1"/>
 <contactref element="R2" pad="2"/>
@@
 <wire x1="15.24" y1="16.8275" x2="17.145" y2="18.7325" width="0.3048" layer="1"/>
 <wire x1="17.145" y1="18.7325" x2="17.4625" y2="18.7325" width="0.3048" layer="1"/>
+<wire x1="7.46125" y1="41.75125" x2="7.46125" y2="25.4" width="1.27" layer="1"/>
+<wire x1="11.1125" y1="45.4025" x2="7.46125" y2="41.75125" width="1.27" layer="1"/>
+<wire x1="11.1125" y1="45.4025" x2="11.1125" y2="50.4825" width="1.27" layer="1"/>
 <contactref element="D1" pad="C"/>
-<wire x1="8.8425" y1="42.91" x2="8.73125" y2="43.02125" width="0.8128" layer="1"/>
-<wire x1="8.8425" y1="42.91" x2="8.8425" y2="24.01875" width="1.27" layer="1"/>
-<wire x1="11.1125" y1="45.4025" x2="8.73125" y2="43.02125" width="1.27" layer="1"/>
-<wire x1="11.1125" y1="45.4025" x2="11.1125" y2="50.4825" width="1.27" layer="1"/>
-<wire x1="5.3975" y1="43.18" x2="8.5725" y2="43.18" width="1.27" layer="1"/>
-<wire x1="11.1125" y1="50.4825" x2="8.5725" y2="43.18" width="0" layer="19" extent="1-1"/>
+<wire x1="5.3975" y1="42.8625" x2="6.35" y2="42.8625" width="1.27" layer="1"/>
+<wire x1="6.35" y1="42.8625" x2="7.46125" y2="41.75125" width="1.27" layer="1"/>
 </signal>
 <signal name="5V">
@@
 <contactref element="ARMA" pad="2"/>
 <contactref element="ARMA3" pad="2"/>
-<contactref element="E1" pad="2"/>
+<contactref element="BAT1" pad="2"/>
 <polygon width="0.8128" layer="1" isolate="0.6096">
 <vertex x="0" y="0.3175"/>
@@
 </signal>
 <signal name="N$2">
-<contactref element="D1" pad="A"/>
-<wire x1="5.3975" y1="50.8" x2="5.3975" y2="54.245" width="1.27" layer="1"/>
 <contactref element="ARMA3" pad="1"/>
-<contactref element="E1" pad="1"/>
+<contactref element="BAT1" pad="1"/>
 <wire x1="5.3975" y1="54.245" x2="12.9239" y2="61.7714" width="1.27" layer="1"/>
 <wire x1="20.995" y1="58.42" x2="17.6436" y2="61.7714" width="1.27" layer="1"/>
@@
 <wire x1="14.2875" y1="61.7714" x2="12.9239" y2="61.7714" width="1.27" layer="1"/>
 <wire x1="14.2875" y1="61.9125" x2="14.2875" y2="61.7714" width="0.8128" layer="1"/>
+<contactref element="D1" pad="A"/>
+<wire x1="5.3975" y1="50.4825" x2="5.3975" y2="54.245" width="1.27" layer="1"/>
 </signal>
 <signal name="N$19">
